File: KicadFiles/Non-LED/900Than9.kicad_pcb (KiCad board)
At the start: 2 copper layers, 356.9 x 129.1 mm, 264 parts, among them J1 Conn_01x04_Pin, J2 USB_C_Receptacle_USB2.0_14P, SW1 SW_Reset, SW2 SW_Boot, U1 XC6206PxxxMR, U2 RP2040, U3 SRV05-4, U4 W25Q128JVS, Y1 ABM8-272-T3

Commit message: Updated LED placement & footprints
Parts:
- C1, C10, C11, C12, C13, C14, C15, C16, C17, C18, C2, C3, C4, C5, C6, C7, C8, C9, F1, J1, J2, R1, R2, R3, R4, R5, R6, R7, R8, R9, SW1, SW2, U1, U2, U3, U4, Y1: moved to B.Cu
- LED1, LED2: footprint PCM_marbastlib-mx:LED_MX_3mm -> My-Fi Footprints:DIP_LED_MX_3mm
- moved LED1 642.0 mm to (27.5, 27.4)
- moved LED3 590.5 mm to (34.7, 89.3)
- moved C1 432.0 mm to (293.0, 206.4)
- moved C15 432.0 mm to (298.7, 206.4)
- moved C8 432.0 mm to (295.9, 206.4)
- moved C16 430.6 mm to (298.7, 204.4)
- moved C2 430.6 mm to (293.0, 204.4)
- moved C9 430.6 mm to (295.9, 204.4)
- moved SW1 430.4 mm to (304.4, 204.0)
- moved U4 430.2 mm to (324.5, 178.1)
- moved C10 429.3 mm to (295.9, 202.4)
- moved C17 429.3 mm to (298.7, 202.4)
- moved C3 429.3 mm to (293.0, 202.4)
- moved J2 428.7 mm to (314.6, 201.5)
- moved C11 428.0 mm to (295.9, 200.4)
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
Commit message: Update 900Than9.kicad_pcb
Parts:
- removed C10, C11, C12, C14, C15, C16: 100n, Capacitor_SMD:C_0402_1005Metric
- removed C13: 4.7n, Capacitor_SMD:C_0402_1005Metric
- removed C17, C18: 1u, Capacitor_SMD:C_0402_1005Metric
- removed J2: USB_C_Receptacle_USB2.0_14P, Connector_USB:USB_C_Receptacle_HRO_TYPE-C-31-M-12
- removed R6: 1M, Resistor_SMD:R_0402_1005Metric
- removed R7: 1K, Resistor_SMD:R_0402_1005Metric
- removed R8: 10k, Resistor_SMD:R_0402_1005Metric
- removed R9: 1k, Resistor_SMD:R_0402_1005Metric
- removed U4: W25Q128JVS, My-Fi Footprints:SOIC-8_5.23x5.23mm_P1.27mm
- removed Y1: ABM8-272-T3, My-Fi Footprints:Oscillator_SMD_EuroQuartz_XO32-4Pin_3.2x2.5mm
- added LED4: LED, My-Fi Footprints:DIP_LED_MX_3mm, F.Cu at (32.3, 127.4)
- C1: value 1uF -> 4.7n
- C2: value 1uF -> 100nF
- C3, C4: value 15p -> 100nF
- C5, C6: value 100n -> 100nF
- C7: value 100n -> 10uF
- C8, C9: value 100n -> 1uF
- R1: value 27.4 -> 1M
- R2: value 27.4 -> 220
- R3, R4: value 5.1K -> 220
- R5: value 1K -> 10k
- SW1: value SW_Reset -> SW_DPST_x2
- SW2: value SW_Boot -> SW_DPST_x2
- U1: value XC6206PxxxMR -> SRV05-4; footprint Package_TO_SOT_SMD:SOT-23-3 -> Package_TO_SOT_SMD:SOT-23-6
- U2: value RP2040 -> STM32F072CBTx; footprint My-Fi Footprints:RP2040-QFN-56 -> Package_QFP:LQFP-48_7x7mm_P0.5mm
- U3: value SRV05-4 -> XC6206PxxxMR; footprint Package_TO_SOT_SMD:SOT-23-6 -> Package_TO_SOT_SMD:SOT-23-3
- moved C1 205.0 mm to (464.5, 94.0)
- moved C2 205.0 mm to (464.5, 92.0)
- moved C3 205.0 mm to (464.5, 90.0)
- moved C4 205.0 mm to (464.5, 88.1)
- moved C5 205.0 mm to (464.5, 86.1)
- moved C6 205.0 mm to (464.5, 84.1)
- moved C7 205.0 mm to (464.5, 82.2)
- moved C8 205.0 mm to (467.4, 94.0)
- moved C9 205.0 mm to (467.4, 92.0)
- moved F1 205.0 mm to (494.6, 73.5)
- moved J1 205.0 mm to (487.4, 77.4)
- moved R1 205.0 mm to (493.2, 80.2)
- moved R2 205.0 mm to (493.2, 78.2)
- moved R3 205.0 mm to (493.2, 76.2)
- moved SW1 205.0 mm to (475.9, 91.6)
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Connections:
- C1 pad 1: +5V -> GNDREF
- C2 pad 1: +3V3 -> RST-1
- C3 pad 1: GND -> +3V3
- C3 pad 2: XTAL_IN -> GND
- C4 pad 1: GND -> +3V3
- C4 pad 2: Net-(C4-Pad2) -> GND
- C5 pad 1: GND -> +3V3
- C5 pad 2: +3V3 -> GND
- C6 pad 1: GND -> +3V3
- C6 pad 2: +3V3 -> GND
- C7 pad 1: GND -> +3V3
- C7 pad 2: +3V3 -> GND
- C8 pad 1: GND -> +5V
- C8 pad 2: +3V3 -> GND
- C9 pad 1: GND -> +3V3
- C9 pad 2: +3V3 -> GND
- LED1 pad 1: ESCLED -> Net-(LED1-K)
- LED2 pad 1: SCLLED -> Net-(LED2-K)
- LED3 pad 1: CAPLED -> Net-(LED3-K)
- R1 pad 1: DP -> GNDREF
- R1 pad 2: Net-(U2-USB_DP) -> GND
- R2 pad 1: Net-(U2-USB_DM) -> ESCLED
- R2 pad 2: DN -> Net-(LED1-K)
- R3 pad 1: GND -> SCLLED
- R3 pad 2: Net-(J2-CC2) -> Net-(LED2-K)
- R4 pad 1: GND -> CAPLED
- R4 pad 2: Net-(J2-CC1) -> Net-(LED3-K)
- R5 pad 1: Net-(C4-Pad2) -> BOOT-1
- R5 pad 2: XTAL_OUT -> GND
- SW1 pad 1: RESET -> RST-1
- SW2 pad 1: GND -> BOOT-1
- SW2 pad 2: Net-(SW2A-B) -> +3V3
- U1 pad 1: GND -> unconnected-(U1-IO1-Pad1)
- U1 pad 2: +3V3 -> GND
- U1 pad 3: +5V -> unconnected-(U1-IO2-Pad3)
- U2 pad 1: Net-(U2-ADC_AVDD) -> +3V3
- U2 pad 10: Net-(U2-ADC_AVDD) -> unconnected-(U2-PA0-Pad10)
- U2 pad 19: GND -> unconnected-(U2-PB1-Pad19)
- U2 pad 20: XTAL_IN -> unconnected-(U2-PB2-Pad20)
- U2 pad 21: XTAL_OUT -> unconnected-(U2-PB10-Pad21)
- U2 pad 22: Net-(U2-ADC_AVDD) -> unconnected-(U2-PB11-Pad22)
- U2 pad 23: Net-(U2-VREG_VOUT) -> GND
- U2 pad 24: SWCLK -> +3V3
- U2 pad 25: SWD -> unconnected-(U2-PB12-Pad25)
- U2 pad 26: RESET -> unconnected-(U2-PB13-Pad26)
- U2 pad 32: unconnected-(U2-GPIO21-Pad32) -> DN
- U2 pad 33: Net-(U2-ADC_AVDD) -> DP
- U2 pad 35: unconnected-(U2-GPIO23-Pad35) -> GND
- U2 pad 36: unconnected-(U2-GPIO24-Pad36) -> +3V3
- U2 pad 42: Net-(U2-ADC_AVDD) -> unconnected-(U2-PB6-Pad42)
- U2 pad 43: Net-(U2-ADC_AVDD) -> unconnected-(U2-PB7-Pad43)
- U2 pad 44: Net-(U2-ADC_AVDD) -> BOOT-1
- U2 pad 45: Net-(U2-VREG_VOUT) -> unconnected-(U2-PB8-Pad45)
- U2 pad 46: Net-(U2-USB_DM) -> unconnected-(U2-PB9-Pad46)
- U2 pad 47: Net-(U2-USB_DP) -> GND
- U2 pad 48: Net-(U2-ADC_AVDD) -> +3V3
- U2 pad 7: unconnected-(U2-GPIO5-Pad7) -> RST-1
- U2 pad 8: unconnected-(U2-GPIO6-Pad8) -> GND
- U2 pad 9: unconnected-(U2-GPIO7-Pad9) -> +3V3
- U3 pad 1: unconnected-(U3-IO1-Pad1) -> GND
- U3 pad 2: GND -> +3V3
- U3 pad 3: unconnected-(U3-IO2-Pad3) -> +5V
Other:
- board size 356.9 x 129.1 mm -> 344.7 x 123.6 mm

Commit message: updated pcb & sch
Parts:
- removed D100, D102, D15, D32, D51, D55, D69, D71, D73, D74, D87, D92, D96, D99: 1N4148, Diode_SMD:D_SOD-323_HandSoldering
- added J2: Conn_01x01_Pin, TestPoint:TestPoint_THTPad_2.0x2.0mm_Drill1.0mm, B.Cu at (303.6, 19.5)
- added Outline1: ~, My-Fi Footprints:A87-outline_jst, F.Cu at (25.0, 25.0)
- MX1, MX10, MX101, MX103, MX104, MX106, MX107, MX108, MX11, MX12, MX13, MX14, MX15, MX16, MX17, MX18, MX19, MX2, MX20, MX21, MX22, MX23, MX24, MX25, MX26, MX27, MX28, MX29, MX3, MX30, MX31, MX32, MX33, MX34, MX35, MX36, MX38, MX39, MX4, MX40, MX41, MX42, MX43, MX44, MX45, MX46, MX47, MX48, MX49, MX5, MX51, MX52, MX53, MX54, MX57, MX58, MX59, MX6, MX60, MX61, MX62, MX63, MX64, MX65, MX66, MX67, MX68, MX69, MX7, MX71, MX73, MX75, MX76, MX77, MX78, MX79, MX8, MX80, MX81, MX82, MX83, MX84, MX85, MX87, MX88, MX89, MX9, MX91, MX92, MX94, MX95, MX96, MX97, MX98, MX99: footprint PCM_marbastlib-mx:SW_MX_1u -> My-Fi Footprints:SW_MX_1u
- MX100, MX102, MX105, MX37, MX50, MX90, MX93: footprint PCM_marbastlib-mx:SW_MX_1.5u -> My-Fi Footprints:SW_MX_1.5u
- MX55: footprint PCM_marbastlib-mx:SW_MX_1.75u_STP_1.25 -> My-Fi Footprints:SW_MX_1.75u_STP_1.25
- MX56, MX86: footprint PCM_marbastlib-mx:SW_MX_1.75u -> My-Fi Footprints:SW_MX_1.75u
- MX70, MX72, MX74: footprint PCM_marbastlib-mx:SW_MX_1.25u -> My-Fi Footprints:SW_MX_1.25u
- moved R2 473.6 mm to (21.9, 32.7), turned to 90 degrees
- moved R4 464.3 mm to (32.1, 94.7), turned to 180 degrees
- moved F1 200.0 mm to (297.9, 37.1), turned to -90 degrees
- moved R1 197.7 mm to (304.4, 22.0), turned to -90 degrees
- moved J1 188.0 mm to (303.6, 37.5)
- moved U1 180.4 mm to (303.5, 43.1), turned to 90 degrees
- moved C1 177.0 mm to (302.8, 22.0), turned to -90 degrees
- moved U3 175.4 mm to (305.1, 79.7), turned to 90 degrees
- moved R3 168.3 mm to (331.4, 30.1), turned to 90 degrees
- moved C9 165.1 mm to (302.6, 81.3), turned to 180 degrees
- moved C8 164.6 mm to (303.6, 78.1), turned to 180 degrees
- moved C3 155.5 mm to (309.0, 86.2), turned to 180 degrees
- moved U2 155.2 mm to (315.3, 89.1), turned to 90 degrees
- moved C7 151.3 mm to (313.8, 95.3), turned to -90 degrees
- moved R5 149.6 mm to (347.1, 91.0)
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Connections:
- D1 pad 1: unconnected-(D1-K-Pad1) -> ROW0
- D10 pad 1: unconnected-(D10-K-Pad1) -> ROW0
- D101 pad 1: unconnected-(D101-K-Pad1) -> ROW5
- D103 pad 1: unconnected-(D103-K-Pad1) -> ROW5
- D104 pad 1: unconnected-(D104-K-Pad1) -> ROW5
- D105 pad 1: unconnected-(D105-K-Pad1) -> ROW5
- D106 pad 1: unconnected-(D106-K-Pad1) -> ROW5
- D107 pad 1: unconnected-(D107-K-Pad1) -> ROW5
- D108 pad 1: unconnected-(D108-K-Pad1) -> ROW5
- D11 pad 1: unconnected-(D11-K-Pad1) -> ROW0
- D12 pad 1: unconnected-(D12-K-Pad1) -> ROW0
- D13 pad 1: unconnected-(D13-K-Pad1) -> ROW0
- D14 pad 1: unconnected-(D14-K-Pad1) -> ROW0
- D16 pad 1: unconnected-(D16-K-Pad1) -> ROW0
- D17 pad 1: unconnected-(D17-K-Pad1) -> ROW0
- D18 pad 1: unconnected-(D18-K-Pad1) -> ROW1
- D19 pad 1: unconnected-(D19-K-Pad1) -> ROW1
- D2 pad 1: unconnected-(D2-K-Pad1) -> ROW0
- D20 pad 1: unconnected-(D20-K-Pad1) -> ROW1
- D21 pad 1: unconnected-(D21-K-Pad1) -> ROW1
- D22 pad 1: unconnected-(D22-K-Pad1) -> ROW1
- D23 pad 1: unconnected-(D23-K-Pad1) -> ROW1
- D24 pad 1: unconnected-(D24-K-Pad1) -> ROW1
- D25 pad 1: unconnected-(D25-K-Pad1) -> ROW1
- D26 pad 1: unconnected-(D26-K-Pad1) -> ROW1
- D27 pad 1: unconnected-(D27-K-Pad1) -> ROW1
- D28 pad 1: unconnected-(D28-K-Pad1) -> ROW1
- D29 pad 1: unconnected-(D29-K-Pad1) -> ROW1
- D3 pad 1: unconnected-(D3-K-Pad1) -> ROW0
- D30 pad 1: unconnected-(D30-K-Pad1) -> ROW1
- D31 pad 1: unconnected-(D31-K-Pad1) -> ROW1
- D33 pad 1: unconnected-(D33-K-Pad1) -> ROW1
- D34 pad 1: unconnected-(D34-K-Pad1) -> ROW1
- D35 pad 1: unconnected-(D35-K-Pad1) -> ROW1
- D36 pad 1: unconnected-(D36-K-Pad1) -> ROW1
- D37 pad 1: unconnected-(D37-K-Pad1) -> ROW2
- D38 pad 1: unconnected-(D38-K-Pad1) -> ROW2
- D39 pad 1: unconnected-(D39-K-Pad1) -> ROW2
- D4 pad 1: unconnected-(D4-K-Pad1) -> ROW0
- D40 pad 1: unconnected-(D40-K-Pad1) -> ROW2
- D41 pad 1: unconnected-(D41-K-Pad1) -> ROW2
- D42 pad 1: unconnected-(D42-K-Pad1) -> ROW2
- D43 pad 1: unconnected-(D43-K-Pad1) -> ROW2
- D44 pad 1: unconnected-(D44-K-Pad1) -> ROW2
- D45 pad 1: unconnected-(D45-K-Pad1) -> ROW2
- D46 pad 1: unconnected-(D46-K-Pad1) -> ROW2
- D47 pad 1: unconnected-(D47-K-Pad1) -> ROW2
- D48 pad 1: unconnected-(D48-K-Pad1) -> ROW2
- D49 pad 1: unconnected-(D49-K-Pad1) -> ROW2
- D5 pad 1: unconnected-(D5-K-Pad1) -> ROW0
- D50 pad 1: unconnected-(D50-K-Pad1) -> ROW2
- D52 pad 1: unconnected-(D52-K-Pad1) -> ROW2
- D53 pad 1: unconnected-(D53-K-Pad1) -> ROW2
- D54 pad 1: unconnected-(D54-K-Pad1) -> ROW2
- D56 pad 1: unconnected-(D56-K-Pad1) -> ROW3
- D57 pad 1: unconnected-(D57-K-Pad1) -> ROW3
- D58 pad 1: unconnected-(D58-K-Pad1) -> ROW3
- D59 pad 1: unconnected-(D59-K-Pad1) -> ROW3
- D6 pad 1: unconnected-(D6-K-Pad1) -> ROW0
- D60 pad 1: unconnected-(D60-K-Pad1) -> ROW3
- D61 pad 1: unconnected-(D61-K-Pad1) -> ROW3
- D62 pad 1: unconnected-(D62-K-Pad1) -> ROW3
- D63 pad 1: unconnected-(D63-K-Pad1) -> ROW3
- D64 pad 1: unconnected-(D64-K-Pad1) -> ROW3
- D65 pad 1: unconnected-(D65-K-Pad1) -> ROW3
- D66 pad 1: unconnected-(D66-K-Pad1) -> ROW3
- D67 pad 1: unconnected-(D67-K-Pad1) -> ROW3
- D68 pad 1: unconnected-(D68-K-Pad1) -> ROW3
- D7 pad 1: unconnected-(D7-K-Pad1) -> ROW0
- D70 pad 1: unconnected-(D70-K-Pad1) -> ROW3
- D72 pad 1: unconnected-(D72-K-Pad1) -> ROW4
- D75 pad 1: unconnected-(D75-K-Pad1) -> ROW4
- D76 pad 1: unconnected-(D76-K-Pad1) -> ROW4
- D77 pad 1: unconnected-(D77-K-Pad1) -> ROW4
- D78 pad 1: unconnected-(D78-K-Pad1) -> ROW4
- D79 pad 1: unconnected-(D79-K-Pad1) -> ROW4
- D8 pad 1: unconnected-(D8-K-Pad1) -> ROW0
- D80 pad 1: unconnected-(D80-K-Pad1) -> ROW4
- D81 pad 1: unconnected-(D81-K-Pad1) -> ROW4
- D82 pad 1: unconnected-(D82-K-Pad1) -> ROW4
- D83 pad 1: unconnected-(D83-K-Pad1) -> ROW4
- D84 pad 1: unconnected-(D84-K-Pad1) -> ROW4
- D85 pad 1: unconnected-(D85-K-Pad1) -> ROW4
- D86 pad 1: unconnected-(D86-K-Pad1) -> ROW4
- D88 pad 1: unconnected-(D88-K-Pad1) -> ROW4
- D89 pad 1: unconnected-(D89-K-Pad1) -> ROW4
- D9 pad 1: unconnected-(D9-K-Pad1) -> ROW0
- D90 pad 1: unconnected-(D90-K-Pad1) -> ROW5
- D91 pad 1: unconnected-(D91-K-Pad1) -> ROW5
- D93 pad 1: unconnected-(D93-K-Pad1) -> ROW5
- D94 pad 1: unconnected-(D94-K-Pad1) -> ROW5
- D95 pad 1: unconnected-(D95-K-Pad1) -> ROW5
- D97 pad 1: unconnected-(D97-K-Pad1) -> ROW5
- D98 pad 1: unconnected-(D98-K-Pad1) -> ROW5
- LED1 pad 1: Net-(LED1-K) -> GND
- LED1 pad 2: GND -> Net-(LED1-A)
- LED2 pad 1: Net-(LED2-K) -> GND
- LED2 pad 2: GND -> Net-(LED2-A)
- LED3 pad 1: Net-(LED3-K) -> GND
- LED3 pad 2: GND -> Net-(LED3-A)
- LED4 pad 1: Net-(LED3-K) -> GND
- LED4 pad 2: GND -> Net-(LED3-A)
- MX1 pad 1: unconnected-(MX1-Pad1) -> COL0
- MX10 pad 1: unconnected-(MX10-Pad1) -> COL11
- MX100 pad 1: unconnected-(MX100-Pad1) -> COL10
- MX100 pad 2: Net-(D100-A) -> Net-(D101-A)
- MX101 pad 1: unconnected-(MX101-Pad1) -> COL10
- MX102 pad 1: unconnected-(MX102-Pad1) -> COL12
- MX102 pad 2: Net-(D102-A) -> Net-(D103-A)
- MX103 pad 1: unconnected-(MX103-Pad1) -> COL12
- MX104 pad 1: unconnected-(MX104-Pad1) -> COL13
- MX105 pad 1: unconnected-(MX105-Pad1) -> COL14
- MX106 pad 1: unconnected-(MX106-Pad1) -> COL15
- MX107 pad 1: unconnected-(MX107-Pad1) -> COL16
- MX108 pad 1: unconnected-(MX108-Pad1) -> COL17
- MX11 pad 1: unconnected-(MX11-Pad1) -> COL12
- MX12 pad 1: unconnected-(MX12-Pad1) -> COL13
- MX13 pad 1: unconnected-(MX13-Pad1) -> COL14
- MX14 pad 1: unconnected-(MX14-Pad1) -> COL15
- MX15 pad 1: unconnected-(MX15-Pad1) -> COL16
- MX15 pad 2: Net-(D15-A) -> Net-(D16-A)
- MX16 pad 1: unconnected-(MX16-Pad1) -> COL16
- MX17 pad 1: unconnected-(MX17-Pad1) -> COL17
- MX18 pad 1: unconnected-(MX18-Pad1) -> COL0
- MX19 pad 1: unconnected-(MX19-Pad1) -> COL1
- MX2 pad 1: unconnected-(MX2-Pad1) -> COL2
- MX20 pad 1: unconnected-(MX20-Pad1) -> COL2
- MX21 pad 1: unconnected-(MX21-Pad1) -> COL3
- MX22 pad 1: unconnected-(MX22-Pad1) -> COL4
- MX23 pad 1: unconnected-(MX23-Pad1) -> COL5
- MX24 pad 1: unconnected-(MX24-Pad1) -> COL6
- MX25 pad 1: unconnected-(MX25-Pad1) -> COL7
- MX26 pad 1: unconnected-(MX26-Pad1) -> COL8
- MX27 pad 1: unconnected-(MX27-Pad1) -> COL9
- MX28 pad 1: unconnected-(MX28-Pad1) -> COL10
- MX29 pad 1: unconnected-(MX29-Pad1) -> COL11
- MX3 pad 1: unconnected-(MX3-Pad1) -> COL3
- MX30 pad 1: unconnected-(MX30-Pad1) -> COL12
- MX31 pad 1: unconnected-(MX31-Pad1) -> COL13
- MX32 pad 1: unconnected-(MX32-Pad1) -> COL14
- MX32 pad 2: Net-(D32-A) -> Net-(D33-A)
- MX33 pad 1: unconnected-(MX33-Pad1) -> COL14
- MX34 pad 1: unconnected-(MX34-Pad1) -> COL15
- MX35 pad 1: unconnected-(MX35-Pad1) -> COL16
- MX36 pad 1: unconnected-(MX36-Pad1) -> COL17
- MX37 pad 1: unconnected-(MX37-Pad1) -> COL0
- MX38 pad 1: unconnected-(MX38-Pad1) -> COL1
- MX39 pad 1: unconnected-(MX39-Pad1) -> COL2
- MX4 pad 1: unconnected-(MX4-Pad1) -> COL4
- MX40 pad 1: unconnected-(MX40-Pad1) -> COL3
- MX41 pad 1: unconnected-(MX41-Pad1) -> COL4
- MX42 pad 1: unconnected-(MX42-Pad1) -> COL5
- MX43 pad 1: unconnected-(MX43-Pad1) -> COL6
- MX44 pad 1: unconnected-(MX44-Pad1) -> COL7
- MX45 pad 1: unconnected-(MX45-Pad1) -> COL8
- MX46 pad 1: unconnected-(MX46-Pad1) -> COL9
- MX47 pad 1: unconnected-(MX47-Pad1) -> COL10
- MX48 pad 1: unconnected-(MX48-Pad1) -> COL11
- MX49 pad 1: unconnected-(MX49-Pad1) -> COL12
- MX5 pad 1: unconnected-(MX5-Pad1) -> COL5
- MX50 pad 1: unconnected-(MX50-Pad1) -> COL13
- MX51 pad 1: unconnected-(MX51-Pad1) -> COL14
- MX51 pad 2: Net-(D51-A) -> Net-(D70-A)
- MX52 pad 1: unconnected-(MX52-Pad1) -> COL15
- MX53 pad 1: unconnected-(MX53-Pad1) -> COL16
- MX54 pad 1: unconnected-(MX54-Pad1) -> COL17
- MX55 pad 1: unconnected-(MX55-Pad1) -> COL0
- MX55 pad 2: Net-(D55-A) -> Net-(D56-A)
- MX56 pad 1: unconnected-(MX56-Pad1) -> COL0
- MX57 pad 1: unconnected-(MX57-Pad1) -> COL2
- MX58 pad 1: unconnected-(MX58-Pad1) -> COL3
- MX59 pad 1: unconnected-(MX59-Pad1) -> COL4
- MX6 pad 1: unconnected-(MX6-Pad1) -> COL6
- MX60 pad 1: unconnected-(MX60-Pad1) -> COL5
- MX61 pad 1: unconnected-(MX61-Pad1) -> COL6
- MX62 pad 1: unconnected-(MX62-Pad1) -> COL7
- MX63 pad 1: unconnected-(MX63-Pad1) -> COL8
- MX64 pad 1: unconnected-(MX64-Pad1) -> COL9
- MX65 pad 1: unconnected-(MX65-Pad1) -> COL10
- MX66 pad 1: unconnected-(MX66-Pad1) -> COL11
- MX67 pad 1: unconnected-(MX67-Pad1) -> COL12
- MX68 pad 1: unconnected-(MX68-Pad1) -> COL13
- MX69 pad 1: unconnected-(MX69-Pad1) -> COL14
- MX69 pad 2: Net-(D69-A) -> Net-(D70-A)
- MX7 pad 1: unconnected-(MX7-Pad1) -> COL7
- MX70 pad 1: unconnected-(MX70-Pad1) -> COL14
- MX71 pad 1: unconnected-(MX71-Pad1) -> COL0
- MX71 pad 2: Net-(D71-A) -> Net-(D72-A)
- MX72 pad 1: unconnected-(MX72-Pad1) -> COL0
- MX73 pad 1: unconnected-(MX73-Pad1) -> COL1
- MX73 pad 2: Net-(D73-A) -> Net-(D75-A)
- MX74 pad 1: unconnected-(MX74-Pad1) -> COL1
- MX74 pad 2: Net-(D74-A) -> Net-(D75-A)
- MX75 pad 1: unconnected-(MX75-Pad1) -> COL1
- MX76 pad 1: unconnected-(MX76-Pad1) -> COL2
- MX77 pad 1: unconnected-(MX77-Pad1) -> COL3
- MX78 pad 1: unconnected-(MX78-Pad1) -> COL4
- MX79 pad 1: unconnected-(MX79-Pad1) -> COL5
- MX8 pad 1: unconnected-(MX8-Pad1) -> COL8
- MX80 pad 1: unconnected-(MX80-Pad1) -> COL6
- MX81 pad 1: unconnected-(MX81-Pad1) -> COL7
- MX82 pad 1: unconnected-(MX82-Pad1) -> COL8
- MX83 pad 1: unconnected-(MX83-Pad1) -> COL9
- MX84 pad 1: unconnected-(MX84-Pad1) -> COL10
- MX85 pad 1: unconnected-(MX85-Pad1) -> COL11
- MX86 pad 1: unconnected-(MX86-Pad1) -> COL13
- MX87 pad 1: unconnected-(MX87-Pad1) -> COL14
- MX87 pad 2: Net-(D87-A) -> Net-(D88-A)
- MX88 pad 1: unconnected-(MX88-Pad1) -> COL14
- MX89 pad 1: unconnected-(MX89-Pad1) -> COL16
- MX9 pad 1: unconnected-(MX9-Pad1) -> COL9
- MX90 pad 1: unconnected-(MX90-Pad1) -> COL0
- MX91 pad 1: unconnected-(MX91-Pad1) -> COL1
- MX92 pad 1: unconnected-(MX92-Pad1) -> COL2
- MX92 pad 2: Net-(D92-A) -> Net-(D93-A)
- MX93 pad 1: unconnected-(MX93-Pad1) -> COL2
- MX94 pad 1: unconnected-(MX94-Pad1) -> COL3
- MX95 pad 1: unconnected-(MX95-Pad1) -> COL5
- MX96 pad 1: unconnected-(MX96-Pad1) -> COL7
- MX96 pad 2: Net-(D96-A) -> Net-(D97-A)
- MX97 pad 1: unconnected-(MX97-Pad1) -> COL7
- MX98 pad 1: unconnected-(MX98-Pad1) -> COL9
- MX99 pad 1: unconnected-(MX99-Pad1) -> COL10
- MX99 pad 2: Net-(D99-A) -> Net-(D101-A)
- R2 pad 2: Net-(LED1-K) -> Net-(LED1-A)
- R3 pad 2: Net-(LED2-K) -> Net-(LED2-A)
- R4 pad 2: Net-(LED3-K) -> Net-(LED3-A)
Routing:
- net Net-(LED3-A): track 0.00 -> 55.7 mm
- net DN: track 0.00 -> 51.8 mm
- net DP: track 0.00 -> 50.6 mm
- net +5V: track 0.00 -> 49.0 mm, vias 0 -> 4
- net RST-1: track 0.00 -> 48.1 mm
- net +3V3: track 0.00 -> 47.0 mm
- net BOOT-1: track 0.00 -> 38.3 mm
- net GND: track 0.00 -> 37.1 mm
- net Net-(D16-A): track 0.00 -> 18.8 mm
- net Net-(D88-A): track 0.00 -> 16.7 mm
- net COL14: track 0.00 -> 16.7 mm
- net Net-(D70-A): track 0.00 -> 13.5 mm
- net Net-(D75-A): track 0.00 -> 11.9 mm
- net Net-(D33-A): track 0.00 -> 9.53 mm
- net Net-(D101-A): track 0.00 -> 9.53 mm
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Other:
- board size 344.7 x 123.6 mm -> 344.7 x 116.6 mm
