File: KicadFiles/Non-LED/900Than9.kicad_sch (KiCad schematic)
At the start: 264 parts, among them J1 Conn_01x04_Pin, J2 USB_C_Receptacle_USB2.0_14P, SW1 SW_Reset, SW2 SW_Boot, U1 XC6206PxxxMR, U2 RP2040, U3 SRV05-4, U4 W25Q128JVS, Y1 ABM8-272-T3

Commit message: Updated LED placement & footprints
Parts:
- LED1, LED2: footprint PCM_marbastlib-mx:LED_MX_3mm -> My-Fi Footprints:DIP_LED_MX_3mm
Changed lines of the file:
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@@
 			)
 		)
-		(property "Footprint" "PCM_marbastlib-mx:LED_MX_3mm"
+		(property "Footprint" "My-Fi Footprints:DIP_LED_MX_3mm"
 			(at 284.48 237.49 0)
 			(effects
@@
 			)
 		)
-		(property "Footprint" "PCM_marbastlib-mx:LED_MX_3mm"
+		(property "Footprint" "My-Fi Footprints:DIP_LED_MX_3mm"
 			(at 284.48 256.54 0)
 			(effects

Commit message: Update 900Than9.kicad_sch
Other:
- note added: "ISO"
- moved on the sheet: C1, C10, C11, C12, C13, C14, C15, C16, C17, C18, C2, C3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

Commit message: Update 900Than9.kicad_sch
Parts:
- removed C1: 1uF, Capacitor_SMD:C_0402_1005Metric, symbol Device:C
- removed C10, C11, C12, C14, C15, C16, C5, C6, C7, C8, C9: 100n, Capacitor_SMD:C_0402_1005Metric, symbol Device:C_Small
- removed C17, C18: 1u, Capacitor_SMD:C_0402_1005Metric, symbol Device:C_Small
- removed C3, C4: 15p, Capacitor_SMD:C_0402_1005Metric, symbol Device:C_Small
- removed J2: USB_C_Receptacle_USB2.0_14P, Connector_USB:USB_C_Receptacle_HRO_TYPE-C-31-M-12, symbol Connector:USB_C_Receptacle_USB2.0_14P
- removed R1: 27.4, Resistor_SMD:R_0402_1005Metric, symbol Device:R_Small
- removed R5, R7: 1K, Resistor_SMD:R_0402_1005Metric, symbol Device:R_Small
- removed R8: 10k, Resistor_SMD:R_0402_1005Metric, symbol Device:R_Small
- removed R9: 1k, Resistor_SMD:R_0402_1005Metric, symbol Device:R_Small
- removed U2: RP2040, My-Fi Footprints:RP2040-QFN-56, symbol MCU_RaspberryPi_and_Boards:RP2040
- removed U4: W25Q128JVS, My-Fi Footprints:SOIC-8_5.23x5.23mm_P1.27mm, symbol Memory_Flash:W25Q128JVS
- removed Y1: ABM8-272-T3, My-Fi Footprints:Oscillator_SMD_EuroQuartz_XO32-4Pin_3.2x2.5mm, symbol Device:Crystal_GND24
- added C3, C4, C5, C6: 100nF, Capacitor_SMD:C_0402_1005Metric, symbol Device:C
- added C7: 10uF, Capacitor_SMD:C_0402_1005Metric, symbol Device:C
- added C8, C9: 1uF, Capacitor_SMD:C_0402_1005Metric, symbol Device:C
- added LED4: LED, My-Fi Footprints:DIP_LED_MX_3mm, symbol Device:LED
- added R5: 10k, Resistor_SMD:R_0402_1005Metric, symbol Device:R
- added U2: STM32F072CBTx, Package_QFP:LQFP-48_7x7mm_P0.5mm, symbol MCU_ST_STM32F0:STM32F072CBTx
- C2: value 1uF -> 100nF
- R2: value 27.4 -> 220
- R3, R4: value 5.1K -> 220
- SW1: value SW_Reset -> SW_DPST_x2
- SW2: value SW_Boot -> SW_DPST_x2
- renumbered C13 to C1, R6 to R1, U3 to U1, U1 to U3
Connections:
- net +3V3: now also SW2.2 (B), C3.1, C4.1, C5.1, C6.1, C7.1, C9.1, U2.1 (VBAT), U2.24 (VDD), U2.36 (VDDIO2), U2.48 (VDD), U2.9 (VDDA); no longer C2.1
- net +5V: now also C8.1
- net CAPLED: now also R4.1; no longer LED3.1 (K)
- net DN: now also U2.32 (PA11); no longer R2.2
- net DP: now also U2.33 (PA12)
- net ESCLED: now also R2.1; no longer LED1.1 (K)
- net GND: now also C3.2, C4.2, C5.2, C6.2, C7.2, C8.2, C9.2, LED4.2 (A), R5.2, U2.23 (VSS), U2.35 (VSS), U2.47 (VSS), U2.8 (VSSA); no longer R3.1, R4.1, SW2.1 (A)
- net SCLLED: now also R3.1; no longer LED2.1 (K)
- net at R4.2: now also LED3.1 (K), LED4.1 (K)
- net at R3.2: now also LED2.1 (K)
- net RESET renamed RST-1
- net RST-1: now also C2.1, U2.7 (NRST)
- new net: LED1.1 (K), R2.2
- new net BOOT-1: R5.1, SW2.1 (A), U2.44 (BOOT0)
- no-connect marks 2 -> 3
Other:
- note added: "Boot Switch"
- note added: "Decoupling Capacitors"
- note added: "MCU STM32F072CBT6"
- note added: "Regulator XC6206 5V-3.3V"
- note removed: "+1V1, 1uF Cap to Pin 45"
- note removed: "+3V3, 1uF Cap to Pin 44"
- note removed: "Crystal"
- note removed: "Decoupling Capacitor"
- note removed: "Flash"
- note removed: "RP2040"
- note removed: "Regulator"
- note removed: "USB-C"
- moved on the sheet: C1, F1, J1, LED1, LED2, LED3, R1, U1, U3

Commit message: updated pcb & sch
Parts:
- removed D100, D102, D15, D32, D51, D55, D69, D71, D73, D74, D87, D92, D96, D99: 1N4148, Diode_SMD:D_SOD-323_HandSoldering, symbol Device:D
- added J2: Conn_01x01_Pin, TestPoint:TestPoint_THTPad_2.0x2.0mm_Drill1.0mm, symbol Connector:Conn_01x01_Pin
- added Outline1: ~, My-Fi Footprints:A87-outline_jst, symbol My-Fi Symbols:Outline
- MX1, MX10, MX101, MX103, MX104, MX106, MX107, MX108, MX11, MX12, MX13, MX14, MX15, MX16, MX17, MX18, MX19, MX2, MX20, MX21, MX22, MX23, MX24, MX25, MX26, MX27, MX28, MX29, MX3, MX30, MX31, MX32, MX33, MX34, MX35, MX36, MX38, MX39, MX4, MX40, MX41, MX42, MX43, MX44, MX45, MX46, MX47, MX48, MX49, MX5, MX51, MX52, MX53, MX54, MX57, MX58, MX59, MX6, MX60, MX61, MX62, MX63, MX64, MX65, MX66, MX67, MX68, MX69, MX7, MX71, MX73, MX75, MX76, MX77, MX78, MX79, MX8, MX80, MX81, MX82, MX83, MX84, MX85, MX87, MX88, MX89, MX9, MX91, MX92, MX94, MX95, MX96, MX97, MX98, MX99: footprint PCM_marbastlib-mx:SW_MX_1u -> My-Fi Footprints:SW_MX_1u
- MX100, MX102, MX105, MX37, MX50, MX90, MX93: footprint PCM_marbastlib-mx:SW_MX_1.5u -> My-Fi Footprints:SW_MX_1.5u
- MX55: footprint PCM_marbastlib-mx:SW_MX_1.75u_STP_1.25 -> My-Fi Footprints:SW_MX_1.75u_STP_1.25
- MX56, MX86: footprint PCM_marbastlib-mx:SW_MX_1.75u -> My-Fi Footprints:SW_MX_1.75u
- MX70, MX72, MX74: footprint PCM_marbastlib-mx:SW_MX_1.25u -> My-Fi Footprints:SW_MX_1.25u
Connections:
- net GND: now also LED1.1 (K), LED2.1 (K), LED3.1 (K), LED4.1 (K); no longer LED1.2 (A), LED2.2 (A), LED3.2 (A), LED4.2 (A)
- net GNDREF: now also J2.1 (Pin_1)
- net COL13: now reaches MX50.1
- net COL13: now also MX104.1, MX12.1, MX31.1, MX68.1, MX86.1
- net ROW4: now reaches D85.1 (K)
- net ROW4: now also D72.1 (K), D75.1 (K), D76.1 (K), D77.1 (K), D78.1 (K), D79.1 (K), D80.1 (K), D81.1 (K), D82.1 (K), D83.1 (K), D84.1 (K), D86.1 (K), D88.1 (K), D89.1 (K)
- net COL1: now reaches MX73.1
- net COL1: now also MX19.1, MX38.1, MX74.1, MX75.1, MX91.1
- net at MX73.2: now also D75.2 (A), MX74.2, MX75.2
- net ROW1: now reaches D29.1 (K)
- net ROW1: now also D18.1 (K), D19.1 (K), D20.1 (K), D21.1 (K), D22.1 (K), D23.1 (K), D24.1 (K), D25.1 (K), D26.1 (K), D27.1 (K), D28.1 (K), D30.1 (K), D31.1 (K), D33.1 (K), D34.1 (K), D35.1 (K), D36.1 (K)
- net at MX15.2: now also D16.2 (A), MX16.2
- net at R2.2: now also LED1.2 (A); no longer LED1.1 (K)
- net COL0: now reaches MX90.1
- net COL0: now also MX1.1, MX18.1, MX37.1, MX55.1, MX56.1, MX71.1, MX72.1
- net ROW2: now reaches D40.1 (K)
- net ROW2: now also D37.1 (K), D38.1 (K), D39.1 (K), D41.1 (K), D42.1 (K), D43.1 (K), D44.1 (K), D45.1 (K), D46.1 (K), D47.1 (K), D48.1 (K), D49.1 (K), D50.1 (K), D52.1 (K), D53.1 (K), D54.1 (K)
- net COL8: now reaches MX45.1
- net COL8: now also MX26.1, MX63.1, MX8.1, MX82.1
- net COL9: now reaches MX9.1
- net COL9: now also MX27.1, MX46.1, MX64.1, MX83.1, MX98.1
- net COL14: now reaches MX33.1
- net COL14: now also MX105.1, MX13.1, MX32.1, MX51.1, MX69.1, MX70.1, MX87.1, MX88.1
- net at D33.2 (A), MX33.2: now also MX32.2
- net COL4: now reaches MX41.1
- net COL4: now also MX22.1, MX4.1, MX59.1, MX78.1
- net ROW3: now reaches D59.1 (K)
- net ROW3: now also D56.1 (K), D57.1 (K), D58.1 (K), D60.1 (K), D61.1 (K), D62.1 (K), D63.1 (K), D64.1 (K), D65.1 (K), D66.1 (K), D67.1 (K), D68.1 (K), D70.1 (K)
- net at MX51.2: now also D70.2 (A), MX69.2, MX70.2
- net COL17: now reaches MX36.1
- net COL17: now also MX108.1, MX17.1, MX54.1
- net ROW5: now reaches D101.1 (K)
- net ROW5: now also D103.1 (K), D104.1 (K), D105.1 (K), D106.1 (K), D107.1 (K), D108.1 (K), D90.1 (K), D91.1 (K), D93.1 (K), D94.1 (K), D95.1 (K), D97.1 (K), D98.1 (K)
- net at D101.2 (A), MX101.2: now also MX100.2, MX99.2
- net ROW0: now reaches D12.1 (K)
- net ROW0: now also D1.1 (K), D10.1 (K), D11.1 (K), D13.1 (K), D14.1 (K), D16.1 (K), D17.1 (K), D2.1 (K), D3.1 (K), D4.1 (K), D5.1 (K), D6.1 (K), D7.1 (K), D8.1 (K), D9.1 (K)
- net COL6: now reaches MX6.1
- net COL6: now also MX24.1, MX43.1, MX61.1, MX80.1
- net COL10: now reaches MX100.1
- net COL10: now also MX101.1, MX28.1, MX47.1, MX65.1, MX84.1, MX99.1
- net COL11: now reaches MX29.1
- net COL11: now also MX10.1, MX48.1, MX66.1, MX85.1
- net COL7: now reaches MX25.1
- net COL7: now also MX44.1, MX62.1, MX7.1, MX81.1, MX96.1, MX97.1
- net COL15: now reaches MX34.1
- net COL15: now also MX106.1, MX14.1, MX52.1
- net COL5: now reaches MX79.1
- net COL5: now also MX23.1, MX42.1, MX5.1, MX60.1, MX95.1
- net at D56.2 (A), MX56.2: now also MX55.2
- net COL12: now reaches MX103.1
- net COL12: now also MX102.1, MX11.1, MX30.1, MX49.1, MX67.1
- net at D103.2 (A), MX103.2: now also MX102.2
- net COL2: now reaches MX20.1
- net COL2: now also MX2.1, MX39.1, MX57.1, MX76.1, MX92.1, MX93.1
- net COL16: now reaches MX53.1
- net COL16: now also MX107.1, MX15.1, MX16.1, MX35.1, MX89.1
- net COL3: now reaches MX58.1
- net COL3: now also MX21.1, MX3.1, MX40.1, MX77.1, MX94.1
- net at D88.2 (A), MX88.2: now also MX87.2
- net at MX96.2: now also D97.2 (A), MX97.2
- net at D72.2 (A), MX72.2: now also MX71.2
- net at D93.2 (A), MX93.2: now also MX92.2
- net at R3.2: now also LED2.2 (A); no longer LED2.1 (K)
- new net: LED3.2 (A), LED4.2 (A), R4.2
Other:
- moved on the sheet: D1, D10, D101, D103, D104, D105, D106, D107, D108, D11, D12, D13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

Commit message: first version
Connections:
- net CAPLED: now also U2.18 (PB0)
- net COL0: now also U2.22 (PB11)
- net COL1: now also U2.21 (PB10)
- net COL10: now also U2.25 (PB12)
- net COL11: now also U2.12 (PA2)
- net COL12: now also U2.11 (PA1)
- net COL13: now also U2.6 (PF1)
- net COL14: now also U2.5 (PF0)
- net COL15: now also U2.4 (PC15)
- net COL16: now also U2.3 (PC14)
- net COL17: now also U2.2 (PC13)
- net COL2: now also U2.20 (PB2)
- net COL3: now also U2.19 (PB1)
- net COL4: now also U2.15 (PA5)
- net COL5: now also U2.14 (PA4)
- net COL6: now also U2.13 (PA3)
- net COL7: now also U2.28 (PB15)
- net COL8: now also U2.27 (PB14)
- net COL9: now also U2.26 (PB13)
- net ESCLED: now also U2.16 (PA6)
- net ROW0: now also U2.37 (PA14)
- net ROW1: now also U2.38 (PA15)
- net ROW2: now also U2.39 (PB3)
- net ROW3: now also U2.40 (PB4)
- net ROW4: now also U2.41 (PB5)
- net ROW5: now also U2.42 (PB6)
- net SCLLED: now also U2.17 (PA7)
