File: KicadFiles/Rev2/900Than9.kicad_sch (KiCad schematic)
At the start: 239 parts, among them J1 Conn_01x04_Pin, J2 Conn_01x01_Pin, SW1 SW_DPST_x2, SW2 SW_DPST_x2, U1 SRV05-4, U2 STM32F072CBTx, U3 XC6206PxxxMR

Commit message: Added rev2
Parts:
- removed S97: MX_stab, PCM_marbastlib-mx:STAB_MX_6u, symbol PCM_marbastlib-mx:MX_stab
- Outline1: value ~ -> Outline; footprint My-Fi Footprints:A87-outline_jst -> My-Fi Footprints:Outline-A87_jst
Changed lines of the file:
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@@
 		(dnp no)
 		(property "Reference" "Outline1"
-			(at 265.43 184.15 0)
+			(at 264.16 182.88 0)
 			(effects
 				(font
@@
 			)
 		)
-		(property "Value" "~"
-			(at 266.7 185.42 0)
+		(property "Value" "Outline"
+			(at 264.16 185.42 0)
 			(effects
 				(font
@@
 			)
 		)
-		(property "Footprint" "My-Fi Footprints:A87-outline_jst"
+		(property "Footprint" "My-Fi Footprints:Outline-A87_jst"
 			(at 267.97 185.42 0)
 			(effects
@@
 					(unit 1)
 				)
-			)
-		)
-	)
-	(symbol
-		(lib_id "PCM_marbastlib-mx:MX_stab")
-		(at 160.02 157.48 0)
-		(unit 1)
-		(exclude_from_sim no)
-		(in_bom yes)
-		(on_board yes)
-		(dnp no)
-		(fields_autoplaced yes)
-		(property "Reference" "S97"
-			(at 166.37 156.0829 0)
-			(effects
-				(font
-					(size 1.27 1.27)
-				)
-				(justify left)
-			)
-		)
-		(property "Value" "MX_stab"
-			(at 166.37 158.6229 0)
-			(effects
-				(font
-					(size 1.27 1.27)
-				)
-				(justify left)
-			)
-		)
-		(property "Footprint" "PCM_marbastlib-mx:STAB_MX_6u"
-			(at 160.02 157.48 0)
-			(effects
-				(font
-					(size 1.27 1.27)
-				)
-				(hide yes)
-			)
-		)
-		(property "Datasheet" ""
-			(at 160.02 157.48 0)
-			(effects
-				(font
-					(size 1.27 1.27)
-				)
-				(hide yes)
-			)
-		)
-		(property "Description" "Cherry MX-style stabilizer"
-			(at 160.02 157.48 0)
-			(effects
-				(font
-					(size 1.27 1.27)
-				)
-				(hide yes)
-			)
-		)
-		(instances
-			(project "900Than9"
-				(path "/c9323b67-6e60-43d3-95e0-b7c3373cbf1d"
-					(reference "S97")
-					(unit 1)
-				)
